Commit message: Added ZED and zarm files to dim_cpp and added URDF for devkit with xarm and zed

File: assets/dim_cpp/urdf/include/devkit_base.urdf.xacro (robot description, xacro)
@@ -32,5 +32,5 @@
             <origin xyz="0 0 0" rpy="0 0 0"/>
             <geometry>
-                <mesh filename="dim_cpp/meshes/devkit_base/devkit_base_wheels_parts/devkit_base_wheels_convex_piece_000.obj">
+                <mesh filename="${file_prefix}/meshes/devkit_base/devkit_base_wheels_parts/devkit_base_wheels_convex_piece_000.obj">
                 <drake:declare_convex/>
                 </mesh>
@@ -40,5 +40,5 @@
             <origin xyz="0 0 0" rpy="0 0 0"/>
             <geometry>
-                <mesh filename="dim_cpp/meshes/devkit_base/devkit_base_wheels_parts/devkit_base_wheels_convex_piece_001.obj">
+                <mesh filename="${file_prefix}/meshes/devkit_base/devkit_base_wheels_parts/devkit_base_wheels_convex_piece_001.obj">
                 <drake:declare_convex/>
                 </mesh>
@@ -48,5 +48,5 @@
             <origin xyz="0 0 0" rpy="0 0 0"/>
             <geometry>
-                <mesh filename="dim_cpp/meshes/devkit_base/devkit_base_wheels_parts/devkit_base_wheels_convex_piece_002.obj">
+                <mesh filename="${file_prefix}/meshes/devkit_base/devkit_base_wheels_parts/devkit_base_wheels_convex_piece_002.obj">
                 <drake:declare_convex/>
                 </mesh>
@@ -56,5 +56,5 @@
             <origin xyz="0 0 0" rpy="0 0 0"/>
             <geometry>
-                <mesh filename="dim_cpp/meshes/devkit_base/devkit_base_wheels_parts/devkit_base_wheels_convex_piece_003.obj">
+                <mesh filename="${file_prefix}/meshes/devkit_base/devkit_base_wheels_parts/devkit_base_wheels_convex_piece_003.obj">
                 <drake:declare_convex/>
                 </mesh>
@@ -64,5 +64,5 @@
             <origin xyz="0 0 0" rpy="0 0 0"/>
             <geometry>
-                <mesh filename="dim_cpp/meshes/devkit_base/devkit_base_wheels_parts/devkit_base_wheels_convex_piece_004.obj">
+                <mesh filename="${file_prefix}/meshes/devkit_base/devkit_base_wheels_parts/devkit_base_wheels_convex_piece_004.obj">
                 <drake:declare_convex/>
                 </mesh>
@@ -72,5 +72,5 @@
             <origin xyz="0 0 0" rpy="0 0 0"/>
             <geometry>
-                <mesh filename="dim_cpp/meshes/devkit_base/devkit_base_wheels_parts/devkit_base_wheels_convex_piece_005.obj">
+                <mesh filename="${file_prefix}/meshes/devkit_base/devkit_base_wheels_parts/devkit_base_wheels_convex_piece_005.obj">
                 <drake:declare_convex/>
                 </mesh>
@@ -80,5 +80,5 @@
             <origin xyz="0 0 0" rpy="0 0 0"/>
             <geometry>
-                <mesh filename="dim_cpp/meshes/devkit_base/devkit_base_wheels_parts/devkit_base_wheels_convex_piece_006.obj">
+                <mesh filename="${file_prefix}/meshes/devkit_base/devkit_base_wheels_parts/devkit_base_wheels_convex_piece_006.obj">
                 <drake:declare_convex/>
                 </mesh>
@@ -88,5 +88,5 @@
             <origin xyz="0 0 0" rpy="0 0 0"/>
             <geometry>
-                <mesh filename="dim_cpp/meshes/devkit_base/devkit_base_wheels_parts/devkit_base_wheels_convex_piece_007.obj">
+                <mesh filename="${file_prefix}/meshes/devkit_base/devkit_base_wheels_parts/devkit_base_wheels_convex_piece_007.obj">
                 <drake:declare_convex/>
                 </mesh>
@@ -96,5 +96,5 @@
             <origin xyz="0 0 0" rpy="0 0 0"/>
             <geometry>
-                <mesh filename="dim_cpp/meshes/devkit_base/devkit_base_wheels_parts/devkit_base_wheels_convex_piece_008.obj">
+                <mesh filename="${file_prefix}/meshes/devkit_base/devkit_base_wheels_parts/devkit_base_wheels_convex_piece_008.obj">
                 <drake:declare_convex/>
                 </mesh>
@@ -104,5 +104,5 @@
             <origin xyz="0 0 0" rpy="0 0 0"/>
             <geometry>
-                <mesh filename="dim_cpp/meshes/devkit_base/devkit_base_wheels_parts/devkit_base_wheels_convex_piece_009.obj">
+                <mesh filename="${file_prefix}/meshes/devkit_base/devkit_base_wheels_parts/devkit_base_wheels_convex_piece_009.obj">
                 <drake:declare_convex/>
                 </mesh>
@@ -112,5 +112,5 @@
             <origin xyz="0 0 0" rpy="0 0 0"/>
             <geometry>
-                <mesh filename="dim_cpp/meshes/devkit_base/devkit_base_wheels_parts/devkit_base_wheels_convex_piece_010.obj">
+                <mesh filename="${file_prefix}/meshes/devkit_base/devkit_base_wheels_parts/devkit_base_wheels_convex_piece_010.obj">
                 <drake:declare_convex/>
                 </mesh>
@@ -120,5 +120,5 @@
             <origin xyz="0 0 0" rpy="0 0 0"/>
             <geometry>
-                <mesh filename="dim_cpp/meshes/devkit_base/devkit_base_wheels_parts/devkit_base_wheels_convex_piece_011.obj">
+                <mesh filename="${file_prefix}/meshes/devkit_base/devkit_base_wheels_parts/devkit_base_wheels_convex_piece_011.obj">
                 <drake:declare_convex/>
                 </mesh>
@@ -128,5 +128,5 @@
             <origin xyz="0 0 0" rpy="0 0 0"/>
             <geometry>
-                <mesh filename="dim_cpp/meshes/devkit_base/devkit_base_wheels_parts/devkit_base_wheels_convex_piece_012.obj">
+                <mesh filename="${file_prefix}/meshes/devkit_base/devkit_base_wheels_parts/devkit_base_wheels_convex_piece_012.obj">
                 <drake:declare_convex/>
                 </mesh>
@@ -136,5 +136,5 @@
             <origin xyz="0 0 0" rpy="0 0 0"/>
             <geometry>
-                <mesh filename="dim_cpp/meshes/devkit_base/devkit_base_wheels_parts/devkit_base_wheels_convex_piece_013.obj">
+                <mesh filename="${file_prefix}/meshes/devkit_base/devkit_base_wheels_parts/devkit_base_wheels_convex_piece_013.obj">
                 <drake:declare_convex/>
                 </mesh>
@@ -144,5 +144,5 @@
             <origin xyz="0 0 0" rpy="0 0 0"/>
             <geometry>
-                <mesh filename="dim_cpp/meshes/devkit_base/devkit_base_wheels_parts/devkit_base_wheels_convex_piece_014.obj">
+                <mesh filename="${file_prefix}/meshes/devkit_base/devkit_base_wheels_parts/devkit_base_wheels_convex_piece_014.obj">
                 <drake:declare_convex/>
                 </mesh>
@@ -152,5 +152,5 @@
             <origin xyz="0 0 0" rpy="0 0 0"/>
             <geometry>
-                <mesh filename="dim_cpp/meshes/devkit_base/devkit_base_wheels_parts/devkit_base_wheels_convex_piece_015.obj">
+                <mesh filename="${file_prefix}/meshes/devkit_base/devkit_base_wheels_parts/devkit_base_wheels_convex_piece_015.obj">
                 <drake:declare_convex/>
                 </mesh>
@@ -160,5 +160,5 @@
             <origin xyz="0 0 0" rpy="0 0 0"/>
             <geometry>
-                <mesh filename="dim_cpp/meshes/devkit_base/devkit_base_wheels_parts/devkit_base_wheels_convex_piece_016.obj">
+                <mesh filename="${file_prefix}/meshes/devkit_base/devkit_base_wheels_parts/devkit_base_wheels_convex_piece_016.obj">
                 <drake:declare_convex/>
                 </mesh>
@@ -168,5 +168,5 @@
             <origin xyz="0 0 0" rpy="0 0 0"/>
             <geometry>
-                <mesh filename="dim_cpp/meshes/devkit_base/devkit_base_wheels_parts/devkit_base_wheels_convex_piece_017.obj">
+                <mesh filename="${file_prefix}/meshes/devkit_base/devkit_base_wheels_parts/devkit_base_wheels_convex_piece_017.obj">
                 <drake:declare_convex/>
                 </mesh>
@@ -176,5 +176,5 @@
             <origin xyz="0 0 0" rpy="0 0 0"/>
             <geometry>
-                <mesh filename="dim_cpp/meshes/devkit_base/devkit_base_wheels_parts/devkit_base_wheels_convex_piece_018.obj">
+                <mesh filename="${file_prefix}/meshes/devkit_base/devkit_base_wheels_parts/devkit_base_wheels_convex_piece_018.obj">
                 <drake:declare_convex/>
                 </mesh>
@@ -184,5 +184,5 @@
             <origin xyz="0 0 0" rpy="0 0 0"/>
             <geometry>
-                <mesh filename="dim_cpp/meshes/devkit_base/devkit_base_wheels_parts/devkit_base_wheels_convex_piece_019.obj">
+                <mesh filename="${file_prefix}/meshes/devkit_base/devkit_base_wheels_parts/devkit_base_wheels_convex_piece_019.obj">
                 <drake:declare_convex/>
                 </mesh>
@@ -192,5 +192,5 @@
             <origin xyz="0 0 0" rpy="0 0 0"/>
             <geometry>
-                <mesh filename="dim_cpp/meshes/devkit_base/devkit_base_wheels_parts/devkit_base_wheels_convex_piece_020.obj">
+                <mesh filename="${file_prefix}/meshes/devkit_base/devkit_base_wheels_parts/devkit_base_wheels_convex_piece_020.obj">
                 <drake:declare_convex/>
                 </mesh>
@@ -200,5 +200,5 @@
             <origin xyz="0 0 0" rpy="0 0 0"/>
             <geometry>
-                <mesh filename="dim_cpp/meshes/devkit_base/devkit_base_wheels_parts/devkit_base_wheels_convex_piece_021.obj">
+                <mesh filename="${file_prefix}/meshes/devkit_base/devkit_base_wheels_parts/devkit_base_wheels_convex_piece_021.obj">
                 <drake:declare_convex/>
                 </mesh>
@@ -208,5 +208,5 @@
             <origin xyz="0 0 0" rpy="0 0 0"/>
             <geometry>
-                <mesh filename="dim_cpp/meshes/devkit_base/devkit_base_wheels_parts/devkit_base_wheels_convex_piece_022.obj">
+                <mesh filename="${file_prefix}/meshes/devkit_base/devkit_base_wheels_parts/devkit_base_wheels_convex_piece_022.obj">
                 <drake:declare_convex/>
                 </mesh>
@@ -216,5 +216,5 @@
             <origin xyz="0 0 0" rpy="0 0 0"/>
             <geometry>
-                <mesh filename="dim_cpp/meshes/devkit_base/devkit_base_wheels_parts/devkit_base_wheels_convex_piece_023.obj">
+                <mesh filename="${file_prefix}/meshes/devkit_base/devkit_base_wheels_parts/devkit_base_wheels_convex_piece_023.obj">
                 <drake:declare_convex/>
                 </mesh>
@@ -224,5 +224,5 @@
             <origin xyz="0 0 0" rpy="0 0 0"/>
             <geometry>
-                <mesh filename="dim_cpp/meshes/devkit_base/devkit_base_wheels_parts/devkit_base_wheels_convex_piece_024.obj">
+                <mesh filename="${file_prefix}/meshes/devkit_base/devkit_base_wheels_parts/devkit_base_wheels_convex_piece_024.obj">
                 <drake:declare_convex/>
                 </mesh>
@@ -232,5 +232,5 @@
             <origin xyz="0 0 0" rpy="0 0 0"/>
             <geometry>
-                <mesh filename="dim_cpp/meshes/devkit_base/devkit_base_wheels_parts/devkit_base_wheels_convex_piece_025.obj">
+                <mesh filename="${file_prefix}/meshes/devkit_base/devkit_base_wheels_parts/devkit_base_wheels_convex_piece_025.obj">
                 <drake:declare_convex/>
                 </mesh>
@@ -240,5 +240,5 @@
             <origin xyz="0 0 0" rpy="0 0 0"/>
             <geometry>
-                <mesh filename="dim_cpp/meshes/devkit_base/devkit_base_wheels_parts/devkit_base_wheels_convex_piece_026.obj">
+                <mesh filename="${file_prefix}/meshes/devkit_base/devkit_base_wheels_parts/devkit_base_wheels_convex_piece_026.obj">
                 <drake:declare_convex/>
                 </mesh>
@@ -248,5 +248,5 @@
             <origin xyz="0 0 0" rpy="0 0 0"/>
             <geometry>
-                <mesh filename="dim_cpp/meshes/devkit_base/devkit_base_wheels_parts/devkit_base_wheels_convex_piece_027.obj">
+                <mesh filename="${file_prefix}/meshes/devkit_base/devkit_base_wheels_parts/devkit_base_wheels_convex_piece_027.obj">
                 <drake:declare_convex/>
                 </mesh>
@@ -256,5 +256,5 @@
             <origin xyz="0 0 0" rpy="0 0 0"/>
             <geometry>
-                <mesh filename="dim_cpp/meshes/devkit_base/devkit_base_wheels_parts/devkit_base_wheels_convex_piece_028.obj">
+                <mesh filename="${file_prefix}/meshes/devkit_base/devkit_base_wheels_parts/devkit_base_wheels_convex_piece_028.obj">
                 <drake:declare_convex/>
                 </mesh>
@@ -264,5 +264,5 @@
             <origin xyz="0 0 0" rpy="0 0 0"/>
             <geometry>
-                <mesh filename="dim_cpp/meshes/devkit_base/devkit_base_wheels_parts/devkit_base_wheels_convex_piece_029.obj">
+                <mesh filename="${file_prefix}/meshes/devkit_base/devkit_base_wheels_parts/devkit_base_wheels_convex_piece_029.obj">
                 <drake:declare_convex/>
                 </mesh>
@@ -272,5 +272,5 @@
             <origin xyz="0 0 0" rpy="0 0 0"/>
             <geometry>
-                <mesh filename="dim_cpp/meshes/devkit_base/devkit_base_wheels_parts/devkit_base_wheels_convex_piece_030.obj">
+                <mesh filename="${file_prefix}/meshes/devkit_base/devkit_base_wheels_parts/devkit_base_wheels_convex_piece_030.obj">
                 <drake:declare_convex/>
                 </mesh>
@@ -280,5 +280,5 @@
             <origin xyz="0 0 0" rpy="0 0 0"/>
             <geometry>
-                <mesh filename="dim_cpp/meshes/devkit_base/devkit_base_wheels_parts/devkit_base_wheels_convex_piece_031.obj">
+                <mesh filename="${file_prefix}/meshes/devkit_base/devkit_base_wheels_parts/devkit_base_wheels_convex_piece_031.obj">
                 <drake:declare_convex/>
                 </mesh>
@@ -288,5 +288,5 @@
             <origin xyz="0 0 0" rpy="0 0 0"/>
             <geometry>
-                <mesh filename="dim_cpp/meshes/devkit_base/devkit_base_wheels_parts/devkit_base_wheels_convex_piece_032.obj">
+                <mesh filename="${file_prefix}/meshes/devkit_base/devkit_base_wheels_parts/devkit_base_wheels_convex_piece_032.obj">
                 <drake:declare_convex/>
                 </mesh>
@@ -296,5 +296,5 @@
             <origin xyz="0 0 0" rpy="0 0 0"/>
             <geometry>
-                <mesh filename="dim_cpp/meshes/devkit_base/devkit_base_wheels_parts/devkit_base_wheels_convex_piece_033.obj">
+                <mesh filename="${file_prefix}/meshes/devkit_base/devkit_base_wheels_parts/devkit_base_wheels_convex_piece_033.obj">
                 <drake:declare_convex/>
                 </mesh>
@@ -304,5 +304,5 @@
             <origin xyz="0 0 0" rpy="0 0 0"/>
             <geometry>
-                <mesh filename="dim_cpp/meshes/devkit_base/devkit_base_wheels_parts/devkit_base_wheels_convex_piece_034.obj">
+                <mesh filename="${file_prefix}/meshes/devkit_base/devkit_base_wheels_parts/devkit_base_wheels_convex_piece_034.obj">
                 <drake:declare_convex/>
                 </mesh>
@@ -312,5 +312,5 @@
             <origin xyz="0 0 0" rpy="0 0 0"/>
             <geometry>
-                <mesh filename="dim_cpp/meshes/devkit_base/devkit_base_wheels_parts/devkit_base_wheels_convex_piece_035.obj">
+                <mesh filename="${file_prefix}/meshes/devkit_base/devkit_base_wheels_parts/devkit_base_wheels_convex_piece_035.obj">
                 <drake:declare_convex/>
                 </mesh>
@@ -320,5 +320,5 @@
             <origin xyz="0 0 0" rpy="0 0 0"/>
             <geometry>
-                <mesh filename="dim_cpp/meshes/devkit_base/devkit_base_wheels_parts/devkit_base_wheels_convex_piece_036.obj">
+                <mesh filename="${file_prefix}/meshes/devkit_base/devkit_base_wheels_parts/devkit_base_wheels_convex_piece_036.obj">
                 <drake:declare_convex/>
                 </mesh>
@@ -328,5 +328,5 @@
             <origin xyz="0 0 0" rpy="0 0 0"/>
             <geometry>
-                <mesh filename="dim_cpp/meshes/devkit_base/devkit_base_wheels_parts/devkit_base_wheels_convex_piece_037.obj">
+                <mesh filename="${file_prefix}/meshes/devkit_base/devkit_base_wheels_parts/devkit_base_wheels_convex_piece_037.obj">
                 <drake:declare_convex/>
                 </mesh>
@@ -336,5 +336,5 @@
             <origin xyz="0 0 0" rpy="0 0 0"/>
             <geometry>
-                <mesh filename="dim_cpp/meshes/devkit_base/devkit_base_wheels_parts/devkit_base_wheels_convex_piece_038.obj">
+                <mesh filename="${file_prefix}/meshes/devkit_base/devkit_base_wheels_parts/devkit_base_wheels_convex_piece_038.obj">
                 <drake:declare_convex/>
                 </mesh>
@@ -344,5 +344,5 @@
             <origin xyz="0 0 0" rpy="0 0 0"/>
             <geometry>
-                <mesh filename="dim_cpp/meshes/devkit_base/devkit_base_wheels_parts/devkit_base_wheels_convex_piece_039.obj">
+                <mesh filename="${file_prefix}/meshes/devkit_base/devkit_base_wheels_parts/devkit_base_wheels_convex_piece_039.obj">
                 <drake:declare_convex/>
                 </mesh>
@@ -352,5 +352,5 @@
             <origin xyz="0 0 0" rpy="0 0 0"/>
             <geometry>
-                <mesh filename="dim_cpp/meshes/devkit_base/devkit_base_wheels_parts/devkit_base_wheels_convex_piece_040.obj">
+                <mesh filename="${file_prefix}/meshes/devkit_base/devkit_base_wheels_parts/devkit_base_wheels_convex_piece_040.obj">
                 <drake:declare_convex/>
                 </mesh>
@@ -360,5 +360,5 @@
             <origin xyz="0 0 0" rpy="0 0 0"/>
             <geometry>
-                <mesh filename="dim_cpp/meshes/devkit_base/devkit_base_wheels_parts/devkit_base_wheels_convex_piece_041.obj">
+                <mesh filename="${file_prefix}/meshes/devkit_base/devkit_base_wheels_parts/devkit_base_wheels_convex_piece_041.obj">
                 <drake:declare_convex/>
                 </mesh>
@@ -368,5 +368,5 @@
             <origin xyz="0 0 0" rpy="0 0 0"/>
             <geometry>
-                <mesh filename="dim_cpp/meshes/devkit_base/devkit_base_wheels_parts/devkit_base_wheels_convex_piece_042.obj">
+                <mesh filename="${file_prefix}/meshes/devkit_base/devkit_base_wheels_parts/devkit_base_wheels_convex_piece_042.obj">
                 <drake:declare_convex/>
                 </mesh>
@@ -376,5 +376,5 @@
             <origin xyz="0 0 0" rpy="0 0 0"/>
             <geometry>
-                <mesh filename="dim_cpp/meshes/devkit_base/devkit_base_wheels_parts/devkit_base_wheels_convex_piece_043.obj">
+                <mesh filename="${file_prefix}/meshes/devkit_base/devkit_base_wheels_parts/devkit_base_wheels_convex_piece_043.obj">
                 <drake:declare_convex/>
                 </mesh>
@@ -384,5 +384,5 @@
             <origin xyz="0 0 0" rpy="0 0 0"/>
             <geometry>
-                <mesh filename="dim_cpp/meshes/devkit_base/devkit_base_wheels_parts/devkit_base_wheels_convex_piece_044.obj">
+                <mesh filename="${file_prefix}/meshes/devkit_base/devkit_base_wheels_parts/devkit_base_wheels_convex_piece_044.obj">
                 <drake:declare_convex/>
                 </mesh>
@@ -392,5 +392,5 @@
             <origin xyz="0 0 0" rpy="0 0 0"/>
             <geometry>
-                <mesh filename="dim_cpp/meshes/devkit_base/devkit_base_wheels_parts/devkit_base_wheels_convex_piece_045.obj">
+                <mesh filename="${file_prefix}/meshes/devkit_base/devkit_base_wheels_parts/devkit_base_wheels_convex_piece_045.obj">
                 <drake:declare_convex/>
                 </mesh>
@@ -400,5 +400,5 @@
             <origin xyz="0 0 0" rpy="0 0 0"/>
             <geometry>
-                <mesh filename="dim_cpp/meshes/devkit_base/devkit_base_wheels_parts/devkit_base_wheels_convex_piece_046.obj">
+                <mesh filename="${file_prefix}/meshes/devkit_base/devkit_base_wheels_parts/devkit_base_wheels_convex_piece_046.obj">
                 <drake:declare_convex/>
                 </mesh>
@@ -408,5 +408,5 @@
             <origin xyz="0 0 0" rpy="0 0 0"/>
             <geometry>
-                <mesh filename="dim_cpp/meshes/devkit_base/devkit_base_wheels_parts/devkit_base_wheels_convex_piece_047.obj">
+                <mesh filename="${file_prefix}/meshes/devkit_base/devkit_base_wheels_parts/devkit_base_wheels_convex_piece_047.obj">
                 <drake:declare_convex/>
                 </mesh>
@@ -416,5 +416,5 @@
             <origin xyz="0 0 0" rpy="0 0 0"/>
             <geometry>
-                <mesh filename="dim_cpp/meshes/devkit_base/devkit_base_wheels_parts/devkit_base_wheels_convex_piece_048.obj">
+                <mesh filename="${file_prefix}/meshes/devkit_base/devkit_base_wheels_parts/devkit_base_wheels_convex_piece_048.obj">
                 <drake:declare_convex/>
                 </mesh>
@@ -424,5 +424,5 @@
             <origin xyz="0 0 0" rpy="0 0 0"/>
             <geometry>
-                <mesh filename="dim_cpp/meshes/devkit_base/devkit_base_wheels_parts/devkit_base_wheels_convex_piece_049.obj">
+                <mesh filename="${file_prefix}/meshes/devkit_base/devkit_base_wheels_parts/devkit_base_wheels_convex_piece_049.obj">
                 <drake:declare_convex/>
                 </mesh>
@@ -432,5 +432,5 @@
             <origin xyz="0 0 0" rpy="0 0 0"/>
             <geometry>
-                <mesh filename="dim_cpp/meshes/devkit_base/devkit_base_wheels_parts/devkit_base_wheels_convex_piece_050.obj">
+                <mesh filename="${file_prefix}/meshes/devkit_base/devkit_base_wheels_parts/devkit_base_wheels_convex_piece_050.obj">
                 <drake:declare_convex/>
                 </mesh>
@@ -440,5 +440,5 @@
             <origin xyz="0 0 0" rpy="0 0 0"/>
             <geometry>
-                <mesh filename="dim_cpp/meshes/devkit_base/devkit_base_wheels_parts/devkit_base_wheels_convex_piece_051.obj">
+                <mesh filename="${file_prefix}/meshes/devkit_base/devkit_base_wheels_parts/devkit_base_wheels_convex_piece_051.obj">
                 <drake:declare_convex/>
                 </mesh>
@@ -448,5 +448,5 @@
             <origin xyz="0 0 0" rpy="0 0 0"/>
             <geometry>
-                <mesh filename="dim_cpp/meshes/devkit_base/devkit_base_wheels_parts/devkit_base_wheels_convex_piece_052.obj">
+                <mesh filename="${file_prefix}/meshes/devkit_base/devkit_base_wheels_parts/devkit_base_wheels_convex_piece_052.obj">
                 <drake:declare_convex/>
                 </mesh>
@@ -456,5 +456,5 @@
             <origin xyz="0 0 0" rpy="0 0 0"/>
             <geometry>
-                <mesh filename="dim_cpp/meshes/devkit_base/devkit_base_wheels_parts/devkit_base_wheels_convex_piece_053.obj">
+                <mesh filename="${file_prefix}/meshes/devkit_base/devkit_base_wheels_parts/devkit_base_wheels_convex_piece_053.obj">
                 <drake:declare_convex/>
                 </mesh>
@@ -464,5 +464,5 @@
             <origin xyz="0 0 0" rpy="0 0 0"/>
             <geometry>
-                <mesh filename="dim_cpp/meshes/devkit_base/devkit_base_wheels_parts/devkit_base_wheels_convex_piece_054.obj">
+                <mesh filename="${file_prefix}/meshes/devkit_base/devkit_base_wheels_parts/devkit_base_wheels_convex_piece_054.obj">
                 <drake:declare_convex/>
                 </mesh>
@@ -472,5 +472,5 @@
             <origin xyz="0 0 0" rpy="0 0 0"/>
             <geometry>
-                <mesh filename="dim_cpp/meshes/devkit_base/devkit_base_wheels_parts/devkit_base_wheels_convex_piece_055.obj">
+                <mesh filename="${file_prefix}/meshes/devkit_base/devkit_base_wheels_parts/devkit_base_wheels_convex_piece_055.obj">
                 <drake:declare_convex/>
                 </mesh>
@@ -480,5 +480,5 @@
             <origin xyz="0 0 0" rpy="0 0 0"/>
             <geometry>
-                <mesh filename="dim_cpp/meshes/devkit_base/devkit_base_wheels_parts/devkit_base_wheels_convex_piece_056.obj">
+                <mesh filename="${file_prefix}/meshes/devkit_base/devkit_base_wheels_parts/devkit_base_wheels_convex_piece_056.obj">
                 <drake:declare_convex/>
                 </mesh>
@@ -488,5 +488,5 @@
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