Commit message: Added proper joint state publisher, updated robot state publisher to support mimic joints, and corrected xarm urdf

File: assets/xarm_devkit_base_descr.urdf (robot description, URDF)
Before this commit: robot devkit_base_descr, 32 links, 31 joints
Links:
- link devkit_base_link: geometry collision mesh filename=dim_cpp/meshes/devkit_base/devkit_base_wheels_parts/devkit_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; collision mesh filename=dim_cpp/meshes/devkit_base/devkit_base_wheels_parts/devkit_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
- link left_finger: geometry collision mesh filename=dim_cpp/meshes/gripper/xarm/left_finger.obj; visual mesh filename=dim_cpp/meshes/gripper/xarm/left_finger.obj
- link left_inner_knuckle: geometry collision mesh filename=dim_cpp/meshes/gripper/xarm/left_inner_knuckle.obj; visual mesh filename=dim_cpp/meshes/gripper/xarm/left_inner_knuckle.obj
- link left_outer_knuckle: geometry collision mesh filename=dim_cpp/meshes/gripper/xarm/left_outer_knuckle.obj; visual mesh filename=dim_cpp/meshes/gripper/xarm/left_outer_knuckle.obj
- link link1: geometry collision mesh filename=dim_cpp/meshes/xarm7/visual/link1.obj; visual mesh filename=dim_cpp/meshes/xarm7/visual/link1.obj
- link link2: geometry collision mesh filename=dim_cpp/meshes/xarm7/visual/link2.obj; visual mesh filename=dim_cpp/meshes/xarm7/visual/link2.obj
- link link3: geometry collision mesh filename=dim_cpp/meshes/xarm7/visual/link3.obj; visual mesh filename=dim_cpp/meshes/xarm7/visual/link3.obj
- link link4: geometry collision mesh filename=dim_cpp/meshes/xarm7/visual/link4.obj; visual mesh filename=dim_cpp/meshes/xarm7/visual/link4.obj
- link link5: geometry collision mesh filename=dim_cpp/meshes/xarm7/visual/link5.obj; visual mesh filename=dim_cpp/meshes/xarm7/visual/link5.obj
- link link6: geometry collision mesh filename=dim_cpp/meshes/xarm7/visual/link6.obj; visual mesh filename=dim_cpp/meshes/xarm7/visual/link6.obj
- link link7: geometry collision mesh filename=dim_cpp/meshes/end_tool/collision/end_tool.obj; visual mesh filename=dim_cpp/meshes/xarm7/visual/link7.obj
- link link_base: geometry collision mesh filename=dim_cpp/meshes/xarm7/visual/link_base.obj; visual mesh filename=dim_cpp/meshes/xarm7/visual/link_base.obj
- link pan_tilt_base: geometry collision mesh filename=dim_cpp/meshes/devkit_base/pan_tilt_base_collision.obj scale=1 1 1; visual mesh filename=dim_cpp/meshes/devkit_base/pan_tilt_base_collision.obj scale=1 1 1
- link pan_tilt_head: geometry collision mesh filename=dim_cpp/meshes/devkit_base/pan_tilt_head_collision.obj scale=1 1 1; visual mesh filename=dim_cpp/meshes/devkit_base/pan_tilt_head_collision.obj scale=1 1 1
- link pan_tilt_pan: geometry collision mesh filename=dim_cpp/meshes/devkit_base/pan_tilt_pan_collision.obj scale=1 1 1; visual mesh filename=dim_cpp/meshes/devkit_base/pan_tilt_pan_collision.obj scale=1 1 1
- link pillar_platform: geometry collision mesh filename=dim_cpp/meshes/devkit_base/pillar_platform_collision.obj scale=1 1 1; visual mesh filename=dim_cpp/meshes/devkit_base/pillar_platform_collision.obj scale=1 1 1
- link piper_angled_mount: geometry collision mesh filename=dim_cpp/meshes/devkit_base/piper_angled_mount_collision.obj scale=1 1 1; visual mesh filename=dim_cpp/meshes/devkit_base/piper_angled_mount_collision.obj scale=1 1 1
- link right_finger: geometry collision mesh filename=dim_cpp/meshes/gripper/xarm/right_finger.obj; visual mesh filename=dim_cpp/meshes/gripper/xarm/right_finger.obj
- link right_inner_knuckle: geometry collision mesh filename=dim_cpp/meshes/gripper/xarm/right_inner_knuckle.obj; visual mesh filename=dim_cpp/meshes/gripper/xarm/right_inner_knuckle.obj
- link right_outer_knuckle: geometry collision mesh filename=dim_cpp/meshes/gripper/xarm/right_outer_knuckle.obj; visual mesh filename=dim_cpp/meshes/gripper/xarm/right_outer_knuckle.obj
- link xarm_gripper_base_link: geometry collision mesh filename=dim_cpp/meshes/gripper/xarm/base_link.obj; visual mesh filename=dim_cpp/meshes/gripper/xarm/base_link.obj
- link zed_camera_center: geometry collision mesh filename=dim_cpp/meshes/zedm.obj; visual mesh filename=dim_cpp/meshes/zedm.obj
