Commit message: Initial Drake test script with new URDF, with diff IK and joint control

File: assets/xarm6_openft_gripper.urdf (robot description, URDF)
Before this commit: robot xarm_openft_gripper, 19 links, 18 joints
Links:
- link left_finger: geometry collision mesh filename=dim_cpp/meshes/gripper/xarm/left_finger.obj; visual mesh filename=dim_cpp/meshes/gripper/xarm/left_finger.obj
- link left_inner_knuckle: geometry collision mesh filename=dim_cpp/meshes/gripper/xarm/left_inner_knuckle.obj; visual mesh filename=dim_cpp/meshes/gripper/xarm/left_inner_knuckle.obj
- link left_outer_knuckle: geometry collision mesh filename=dim_cpp/meshes/gripper/xarm/left_outer_knuckle.obj; visual mesh filename=dim_cpp/meshes/gripper/xarm/left_outer_knuckle.obj
- link link1: geometry collision mesh filename=dim_cpp/meshes/xarm6/visual/link1.obj; visual mesh filename=dim_cpp/meshes/xarm6/visual/link1.obj
- link link2: geometry collision mesh filename=dim_cpp/meshes/xarm6/visual/link2.obj; visual mesh filename=dim_cpp/meshes/xarm6/visual/link2.obj
- link link3: geometry collision mesh filename=dim_cpp/meshes/xarm6/visual/link3.obj; visual mesh filename=dim_cpp/meshes/xarm6/visual/link3.obj
- link link4: geometry collision mesh filename=dim_cpp/meshes/xarm6/visual/link4.obj; visual mesh filename=dim_cpp/meshes/xarm6/visual/link4.obj
- link link5: geometry collision mesh filename=dim_cpp/meshes/xarm6/visual/link5.obj; visual mesh filename=dim_cpp/meshes/xarm6/visual/link5.obj
- link link6: geometry collision mesh filename=dim_cpp/meshes/end_tool/collision/end_tool.obj; visual mesh filename=dim_cpp/meshes/xarm6/visual/link6.obj
- link link_base: geometry collision mesh filename=dim_cpp/meshes/xarm6/visual/link_base.obj; visual mesh filename=dim_cpp/meshes/xarm6/visual/link_base.obj
- link link_openft: geometry collision mesh filename=dim_cpp/meshes/openft/openft-xarm-collision.obj scale=0.001 0.001 0.001; visual mesh filename=dim_cpp/meshes/openft/openft-xarm-collision.obj scale=0.001 0.001 0.001
- link right_finger: geometry collision mesh filename=dim_cpp/meshes/gripper/xarm/right_finger.obj; visual mesh filename=dim_cpp/meshes/gripper/xarm/right_finger.obj
- link right_inner_knuckle: geometry collision mesh filename=dim_cpp/meshes/gripper/xarm/right_inner_knuckle.obj; visual mesh filename=dim_cpp/meshes/gripper/xarm/right_inner_knuckle.obj
- link right_outer_knuckle: geometry collision mesh filename=dim_cpp/meshes/gripper/xarm/right_outer_knuckle.obj; visual mesh filename=dim_cpp/meshes/gripper/xarm/right_outer_knuckle.obj
- link xarm_gripper_base_link: geometry collision mesh filename=dim_cpp/meshes/gripper/xarm/base_link.obj; visual mesh filename=dim_cpp/meshes/gripper/xarm/base_link.obj
